File: schematic/rifle-stm32f103ret6-rev1/rifle.sch (KiCad schematic (older format))
At the start: 16 parts

Commit message: Scheme improved, secial shematic elements for nfr24l01 and rfid-rc522 added
Parts:
- removed P?: CONN_4X2, ~, symbol CONN_4X2
- added K?: IR_LASER, ~, symbol CONN_3
- added P?: MicroSD, ~, symbol CONN_9
- added P?: USART1, ~, symbol CONN_4
- added P?: USART2, ~, symbol CONN_4
- added P?: RFID-RC522-MODULE, ~, symbol RFID-RC522-MODULE
- added P?: CONN_4, ~, symbol CONN_4
- added P?: NRF24L01, ~, symbol NRF24L01
- added P?: IR_LED, ~, symbol CONN_2
- added Q? (x4): MOS_N, ~, symbol MOS_N
- added R? (x4): R, ~, symbol R
Connections:
- net labels added: +5V
- wire segments 61 -> 168

Commit message: Micro sd .lib; ready to tracing
Parts:
- removed P?: MicroSD, ~, symbol CONN_9
- added C5: 470uF, ~, symbol CP1
- added K1: Magazine, ~, symbol CONN_3
- added K2: Sound, ~, symbol CONN_3
- added P1: Indication, ~, symbol CONN_5X2
- added P12: CONN_2, ~, symbol CONN_2
- added P2: MICROSD-SDIO, ~, symbol MICROSD-SDIO
- added P4: CONN_5, ~, symbol CONN_5
- added Q1: MOSFET_N, ~, symbol MOSFET_N
- added U2: 5,0 V LDO, ~, symbol LINSTAB-(1-GND/ADJ,2-OUT,3-IN)
- C1: renamed from C?; value 10uF -> 470uF
- gave numbers to parts that had none: 29
Connections:
- wire segments 168 -> 234
Other:
- moved on the sheet: C10, C6, C7, C8, C9

Commit message: About a half of PCB
Parts:
- added P14: Power_in, ~, symbol CONN_2
- added P15: Power_out, ~, symbol CONN_4
- added R?: R, ~, symbol R
Connections:
- net +3.3V: now also P15.2 (P2); no longer C5.1, U2.2 (Out)
- net +5V: now also C5.1, U2.2 (Out), P15.3 (P3)
- net +BATT: now also P14.1 (P1), P15.4 (P4)
- net GND: now also P14.2 (PM), P15.1 (P1)
Changed lines of the file:
@@
 Sheet 1 1
 Title ""
-Date "17 dec 2014"
+Date "18 dec 2014"
 Rev ""
 Comp ""
@@
 $EndComp
 $Comp
-L +3.3V #PWR032
-U 1 1 5491DD9D
-P 4450 6750
-F 0 "#PWR032" H 4450 6710 30  0001 C CNN
-F 1 "+3.3V" H 4450 6860 30  0000 C CNN
-F 2 "" H 4450 6750 60  0000 C CNN
-F 3 "" H 4450 6750 60  0000 C CNN
-	1    4450 6750
-	0    1    1    0
-$EndComp
-$Comp
 L CP1 C5
 U 1 1 5491DDA3
@@
 $EndComp
 $Comp
-L GND #PWR033
+L GND #PWR032
 U 1 1 5491DDAF
 P 4400 7500
-F 0 "#PWR033" H 4400 7500 30  0001 C CNN
+F 0 "#PWR032" H 4400 7500 30  0001 C CNN
 F 1 "GND" H 4400 7430 30  0001 C CNN
 F 2 "" H 4400 7500 60  0000 C CNN
@@
 $EndComp
 $Comp
-L +BATT #PWR034
+L +BATT #PWR033
 U 1 1 5491DDBB
 P 2900 6750
-F 0 "#PWR034" H 2900 6700 20  0001 C CNN
+F 0 "#PWR033" H 2900 6700 20  0001 C CNN
 F 1 "+BATT" H 2900 6850 30  0000 C CNN
 F 2 "" H 2900 6750 60  0000 C CNN
@@
 	3700 7350 3700 7500
 Wire Wire Line
-	4300 6750 4450 6750
+	4300 6750 4550 6750
 Wire Wire Line
 	4400 6900 4400 6750
@@
 $EndComp
 $Comp
-L GND #PWR035
+L GND #PWR034
 U 1 1 5491E3FB
 P 7650 2100
-F 0 "#PWR035" H 7650 2100 30  0001 C CNN
+F 0 "#PWR034" H 7650 2100 30  0001 C CNN
 F 1 "GND" H 7650 2030 30  0001 C CNN
 F 2 "" H 7650 2100 60  0000 C CNN
@@
 	7300 1900 7750 1900
 $Comp
-L +BATT #PWR036
+L +BATT #PWR035
 U 1 1 5491E5D3
 P 7650 1700
-F 0 "#PWR036" H 7650 1650 20  0001 C CNN
+F 0 "#PWR035" H 7650 1650 20  0001 C CNN
 F 1 "+BATT" H 7650 1800 30  0000 C CNN
 F 2 "" H 7650 1700 60  0000 C CNN
@@
 $EndComp
 $Comp
-L GND #PWR037
+L GND #PWR036
 U 1 1 5491F2E2
 P 8250 1400
-F 0 "#PWR037" H 8250 1400 30  0001 C CNN
+F 0 "#PWR036" H 8250 1400 30  0001 C CNN
 F 1 "GND" H 8250 1330 30  0001 C CNN
 F 2 "" H 8250 1400 60  0000 C CNN
@@
 	6850 3400 6850 1250
 $Comp
-L GND #PWR038
+L GND #PWR037
 U 1 1 5491F7A6
 P 6950 1400
-F 0 "#PWR038" H 6950 1400 30  0001 C CNN
+F 0 "#PWR037" H 6950 1400 30  0001 C CNN
 F 1 "GND" H 6950 1330 30  0001 C CNN
 F 2 "" H 6950 1400 60  0000 C CNN
@@
 $EndComp
 $Comp
-L +BATT #PWR039
+L +BATT #PWR038
 U 1 1 5491F8CB
 P 8650 1250
-F 0 "#PWR039" H 8650 1200 20  0001 C CNN
+F 0 "#PWR038" H 8650 1200 20  0001 C CNN
 F 1 "+BATT" H 8650 1350 30  0000 C CNN
 F 2 "" H 8650 1250 60  0000 C CNN
@@
 $EndComp
 $Comp
-L GND #PWR040
+L GND #PWR039
 U 1 1 5491FB09
 P 5800 1600
-F 0 "#PWR040" H 5800 1600 30  0001 C CNN
+F 0 "#PWR039" H 5800 1600 30  0001 C CNN
 F 1 "GND" H 5800 1530 30  0001 C CNN
 F 2 "" H 5800 1600 60  0000 C CNN
@@
 Wire Wire Line
 	6200 1550 6200 1300
+$Comp
+L CONN_2 P14
+U 1 1 54929F23
+P 1150 1350
+F 0 "P14" V 1100 1350 40  0000 C CNN
+F 1 "Power_in" V 1200 1350 40  0000 C CNN
+F 2 "~" H 1150 1350 60  0000 C CNN
+F 3 "~" H 1150 1350 60  0000 C CNN
+	1    1150 1350
+	-1   0    0    -1
+$EndComp
+$Comp
+L GND #PWR040
+U 1 1 54929F32
+P 1600 1550
+F 0 "#PWR040" H 1600 1550 30  0001 C CNN
+F 1 "GND" H 1600 1480 30  0001 C CNN
+F 2 "" H 1600 1550 60  0000 C CNN
+F 3 "" H 1600 1550 60  0000 C CNN
+	1    1600 1550
+	1    0    0    -1
+$EndComp
+$Comp
+L +BATT #PWR041
+U 1 1 54929F41
+P 1600 1150
+F 0 "#PWR041" H 1600 1100 20  0001 C CNN
+F 1 "+BATT" H 1600 1250 30  0000 C CNN
+F 2 "" H 1600 1150 60  0000 C CNN
+F 3 "" H 1600 1150 60  0000 C CNN
+	1    1600 1150
+	1    0    0    -1
+$EndComp
+Wire Wire Line
+	1500 1250 1600 1250
+Wire Wire Line
+	1600 1250 1600 1150
+Wire Wire Line
+	1500 1450 1600 1450
+Wire Wire Line
+	1600 1450 1600 1550
+$Comp
+L +5V #PWR042
+U 1 1 5492AB52
+P 4550 6750
+F 0 "#PWR042" H 4550 6840 20  0001 C CNN
+F 1 "+5V" H 4550 6840 30  0000 C CNN
+F 2 "" H 4550 6750 60  0000 C CNN
+F 3 "" H 4550 6750 60  0000 C CNN
+	1    4550 6750
+	0    1    1    0
+$EndComp
+$Comp
+L GND #PWR043
+U 1 1 5492AE1B
+P 1950 1550
+F 0 "#PWR043" H 1950 1550 30  0001 C CNN
+F 1 "GND" H 1950 1480 30  0001 C CNN
+F 2 "" H 1950 1550 60  0000 C CNN
+F 3 "" H 1950 1550 60  0000 C CNN
+	1    1950 1550
+	1    0    0    -1
+$EndComp
+Wire Wire Line
+	1950 1550 1950 1450
+Wire Wire Line
+	1950 1450 2100 1450
+$Comp
+L +5V #PWR044
+U 1 1 5492AF34
+P 1900 1250
+F 0 "#PWR044" H 1900 1340 20  0001 C CNN
+F 1 "+5V" H 1900 1340 30  0000 C CNN
+F 2 "" H 1900 1250 60  0000 C CNN
+F 3 "" H 1900 1250 60  0000 C CNN
+	1    1900 1250
+	0    -1   -1   0
+$EndComp
+$Comp
+L +3.3V #PWR045
+U 1 1 5492AF4D
+P 1900 1350
+F 0 "#PWR045" H 1900 1310 30  0001 C CNN
+F 1 "+3.3V" H 1900 1460 30  0000 C CNN
+F 2 "" H 1900 1350 60  0000 C CNN
+F 3 "" H 1900 1350 60  0000 C CNN
+	1    1900 1350
+	0    -1   -1   0
+$EndComp
+Wire Wire Line
+	1900 1250 2100 1250
+Wire Wire Line
+	1900 1350 2100 1350
+$Comp
+L CONN_4 P15
+U 1 1 5492B181
+P 2450 1300
+F 0 "P15" V 2400 1300 50  0000 C CNN
+F 1 "Power_out" V 2500 1300 50  0000 C CNN
+F 2 "~" H 2450 1300 60  0000 C CNN
+F 3 "~" H 2450 1300 60  0000 C CNN
+	1    2450 1300
+	1    0    0    1
+$EndComp
+$Comp
+L +BATT #PWR046
+U 1 1 5492B190
+P 2000 1100
+F 0 "#PWR046" H 2000 1050 20  0001 C CNN
+F 1 "+BATT" H 2000 1200 30  0000 C CNN
+F 2 "" H 2000 1100 60  0000 C CNN
+F 3 "" H 2000 1100 60  0000 C CNN
+	1    2000 1100
+	1    0    0    -1
+$EndComp
+Wire Wire Line
+	2000 1100 2000 1150
+Wire Wire Line
+	2000 1150 2100 1150
+$Comp
+L R R?
+U 1 1 5492DE26
+P 2500 6200
+F 0 "R?" V 2580 6200 40  0000 C CNN
+F 1 "R" V 2507 6201 40  0000 C CNN
+F 2 "~" V 2430 6200 30  0000 C CNN
+F 3 "~" H 2500 6200 30  0000 C CNN
+	1    2500 6200
+	0    -1   -1   0
+$EndComp
 $EndSCHEMATC

Commit message: Some more routing
Parts:
- added R10, R12, R6, R7, R8, R9: 0, ~, symbol R
- R5: renamed from R?; value R -> 0
Connections:
- net +3.3V: now also R5.2; no longer P2.4 (Vdd)
- net +BATT: now also R10.1; no longer C1.1, U1.3 (In), U2.3 (In)
- net GND: now also R12.1; no longer P11.1 (GND), P5.1 (P1)
- net at U3.50 (JTDI/SPI3_NSS/I2S3_WS/PA15): now also R8.1; no longer P10.1 (SDA)
- net at U3.51 (PC10/UART4_TX/SDIO_D2): now also R9.2; no longer P2.1 (DAT2)
- net at U3.54 (PD2/TIM3_ETR/UART5_RX/SDIO_CMD): now also R7.2; no longer P2.3 (CMD)
- net at U3.55 (JTDO/SPI3_SCK/I2S3_CK/PB3): now also R6.1; no longer P10.2 (SCK)
- net at R5.1: now also P2.4 (Vdd)
- new net: C1.1, R10.2, U1.3 (In), U2.3 (In)
- new net: P10.1 (SDA), R8.2
- new net: P10.2 (SCK), R6.2
- new net: P11.1 (GND), P5.1 (P1), R12.2
- new net: P2.1 (DAT2), R9.1
- new net: P2.3 (CMD), R7.1
Other:
- moved on the sheet: R5

Commit message: Rwo wires left
Parts:
- added R11, R13, R14: 0, ~, symbol R
Connections:
- net at U3.15 (USART2_RTS/ADC123_IN1/TIM5_CH2/TIM2_CH2/PA1): now also R11.1; no longer Q1.G
- net at U3.39 (PC8/TIM8_CH3/SDIO_D0): now also R13.2; no longer P2.7 (DAT0)
- net at U3.40 (PC9/TIM8_CH4/SDIO_D1): now also R14.2; no longer P2.8 (DAT1/nIRQ)
- new net: P2.7 (DAT0), R13.1
- new net: P2.8 (DAT1/nIRQ), R14.1
- new net: Q1.G, R11.2
Changed lines of the file:
@@
 Sheet 1 1
 Title ""
-Date "18 dec 2014"
+Date "19 dec 2014"
 Rev ""
 Comp ""
@@
 $EndComp
 $Comp
-L +3.3V #PWR020
+L +3.3V #PWR019
 U 1 1 5490BBDA
 P 9300 4700
-F 0 "#PWR020" H 9300 4660 30  0001 C CNN
+F 0 "#PWR019" H 9300 4660 30  0001 C CNN
 F 1 "+3.3V" H 9300 4810 30  0000 C CNN
 F 2 "" H 9300 4700 60  0000 C CNN
@@
 $EndComp
 $Comp
-L GND #PWR021
+L GND #PWR020
 U 1 1 5490C0FA
 P 9000 3400
-F 0 "#PWR021" H 9000 3400 30  0001 C CNN
+F 0 "#PWR020" H 9000 3400 30  0001 C CNN
 F 1 "GND" H 9000 3330 30  0001 C CNN
 F 2 "" H 9000 3400 60  0000 C CNN
@@
 $EndComp
 $Comp
-L GND #PWR022
+L GND #PWR021
 U 1 1 5490C109
 P 9650 3400
-F 0 "#PWR022" H 9650 3400 30  0001 C CNN
+F 0 "#PWR021" H 9650 3400 30  0001 C CNN
 F 1 "GND" H 9650 3330 30  0001 C CNN
 F 2 "" H 9650 3400 60  0000 C CNN
@@
 $EndComp
 $Comp
-L GND #PWR023
+L GND #PWR022
 U 1 1 5490C118
 P 10250 3400
-F 0 "#PWR023" H 10250 3400 30  0001 C CNN
+F 0 "#PWR022" H 10250 3400 30  0001 C CNN
 F 1 "GND" H 10250 3330 30  0001 C CNN
 F 2 "" H 10250 3400 60  0000 C CNN
@@
 $EndComp
 $Comp
-L GND #PWR024
+L GND #PWR023
 U 1 1 5490C127
 P 10850 3400
-F 0 "#PWR024" H 10850 3400 30  0001 C CNN
+F 0 "#PWR023" H 10850 3400 30  0001 C CNN
 F 1 "GND" H 10850 3330 30  0001 C CNN
 F 2 "" H 10850 3400 60  0000 C CNN
@@
 $EndComp
 $Comp
-L +5V #PWR025
+L +5V #PWR024
 U 1 1 5490C3A8
 P 9850 1600
-F 0 "#PWR025" H 9850 1690 20  0001 C CNN
+F 0 "#PWR024" H 9850 1690 20  0001 C CNN
 F 1 "+5V" H 9850 1690 30  0000 C CNN
 F 2 "" H 9850 1600 60  0000 C CNN
@@
 $EndComp
 $Comp
-L +5V #PWR026
+L +5V #PWR025
 U 1 1 5490CABE
 P 8700 1850
-F 0 "#PWR026" H 8700 1940 20  0001 C CNN
+F 0 "#PWR025" H 8700 1940 20  0001 C CNN
 F 1 "+5V" H 8700 1940 30  0000 C CNN
 F 2 "" H 8700 1850 60  0000 C CNN
@@
 $EndComp
 $Comp
-L GND #PWR027
+L GND #PWR026
 U 1 1 5490CBA5
 P 8500 1900
-F 0 "#PWR027" H 8500 1900 30  0001 C CNN
+F 0 "#PWR026" H 8500 1900 30  0001 C CNN
 F 1 "GND" H 8500 1830 30  0001 C CNN
 F 2 "" H 8500 1900 60  0000 C CNN
@@
 $EndComp
 $Comp
-L +3.3V #PWR028
+L +3.3V #PWR027
 U 1 1 5491DA7B
 P 3050 4750
-F 0 "#PWR028" H 3050 4710 30  0001 C CNN
+F 0 "#PWR027" H 3050 4710 30  0001 C CNN
 F 1 "+3.3V" H 3050 4860 30  0000 C CNN
 F 2 "" H 3050 4750 60  0000 C CNN
@@
 $EndComp
 $Comp
-L GND #PWR029
+L GND #PWR028
 U 1 1 5491DB66
 P 3050 5750
-F 0 "#PWR029" H 3050 5750 30  0001 C CNN
+F 0 "#PWR028" H 3050 5750 30  0001 C CNN
 F 1 "GND" H 3050 5680 30  0001 C CNN
 F 2 "" H 3050 5750 60  0000 C CNN
@@
 $EndComp
 $Comp
-L GND #PWR030
+L GND #PWR029
 U 1 1 5491DD97
 P 3700 7500
-F 0 "#PWR030" H 3700 7500 30  0001 C CNN
+F 0 "#PWR029" H 3700 7500 30  0001 C CNN
 F 1 "GND" H 3700 7430 30  0001 C CNN
 F 2 "" H 3700 7500 60  0000 C CNN
@@
 $EndComp
 $Comp
-L GND #PWR031
+L GND #PWR030
 U 1 1 5491DDAF
 P 4400 7500
-F 0 "#PWR031" H 4400 7500 30  0001 C CNN
+F 0 "#PWR030" H 4400 7500 30  0001 C CNN
 F 1 "GND" H 4400 7430 30  0001 C CNN
 F 2 "" H 4400 7500 60  0000 C CNN
@@
 $EndComp
 $Comp
-L +BATT #PWR032
+L +BATT #PWR031
 U 1 1 5491DDBB
 P 2900 6050
-F 0 "#PWR032" H 2900 6000 20  0001 C CNN
+F 0 "#PWR031" H 2900 6000 20  0001 C CNN
 F 1 "+BATT" H 2900 6150 30  0000 C CNN
 F 2 "" H 2900 6050 60  0000 C CNN
@@
 $EndComp
 $Comp
-L GND #PWR033
+L GND #PWR032
 U 1 1 5491E3FB
 P 7650 2100
-F 0 "#PWR033" H 7650 2100 30  0001 C CNN
+F 0 "#PWR032" H 7650 2100 30  0001 C CNN
 F 1 "GND" H 7650 2030 30  0001 C CNN
 F 2 "" H 7650 2100 60  0000 C CNN
@@
 $EndComp
 $Comp
-L +BATT #PWR034
+L +BATT #PWR033
 U 1 1 5491E5D3
 P 7650 1700
-F 0 "#PWR034" H 7650 1650 20  0001 C CNN
+F 0 "#PWR033" H 7650 1650 20  0001 C CNN
 F 1 "+BATT" H 7650 1800 30  0000 C CNN
 F 2 "" H 7650 1700 60  0000 C CNN
@@
 $EndComp
 $Comp
-L GND #PWR035
+L GND #PWR034
 U 1 1 5491F2E2
 P 8250 1400
-F 0 "#PWR035" H 8250 1400 30  0001 C CNN
+F 0 "#PWR034" H 8250 1400 30  0001 C CNN
 F 1 "GND" H 8250 1330 30  0001 C CNN
 F 2 "" H 8250 1400 60  0000 C CNN
@@
 $EndComp
 $Comp
-L GND #PWR036
+L GND #PWR035
 U 1 1 5491F7A6
 P 6950 1400
-F 0 "#PWR036" H 6950 1400 30  0001 C CNN
+F 0 "#PWR035" H 6950 1400 30  0001 C CNN
 F 1 "GND" H 6950 1330 30  0001 C CNN
 F 2 "" H 6950 1400 60  0000 C CNN
@@
 $EndComp
 $Comp
-L +BATT #PWR037
+L +BATT #PWR036
 U 1 1 5491F8CB
 P 8650 1250
-F 0 "#PWR037" H 8650 1200 20  0001 C CNN
+F 0 "#PWR036" H 8650 1200 20  0001 C CNN
 F 1 "+BATT" H 8650 1350 30  0000 C CNN
 F 2 "" H 8650 1250 60  0000 C CNN
@@
 $EndComp
 $Comp
-L GND #PWR038
+L GND #PWR037
 U 1 1 5491FB09
 P 5800 1600
-F 0 "#PWR038" H 5800 1600 30  0001 C CNN
+F 0 "#PWR037" H 5800 1600 30  0001 C CNN
 F 1 "GND" H 5800 1530 30  0001 C CNN
 F 2 "" H 5800 1600 60  0000 C CNN
@@
 $EndComp
 $Comp
-L GND #PWR039
+L GND #PWR038
 U 1 1 54929F32
 P 1600 1550
-F 0 "#PWR039" H 1600 1550 30  0001 C CNN
+F 0 "#PWR038" H 1600 1550 30  0001 C CNN
 F 1 "GND" H 1600 1480 30  0001 C CNN
 F 2 "" H 1600 1550 60  0000 C CNN
@@
 $EndComp
 $Comp
-L +BATT #PWR040
+L +BATT #PWR039
 U 1 1 54929F41
 P 1600 1150
-F 0 "#PWR040" H 1600 1100 20  0001 C CNN
+F 0 "#PWR039" H 1600 1100 20  0001 C CNN
 F 1 "+BATT" H 1600 1250 30  0000 C CNN
 F 2 "" H 1600 1150 60  0000 C CNN
@@
 $EndComp
 $Comp
-L +5V #PWR041
+L +5V #PWR040
 U 1 1 5492AB52
 P 4550 6750
-F 0 "#PWR041" H 4550 6840 20  0001 C CNN
+F 0 "#PWR040" H 4550 6840 20  0001 C CNN
 F 1 "+5V" H 4550 6840 30  0000 C CNN
 F 2 "" H 4550 6750 60  0000 C CNN
@@
 $EndComp
 $Comp
-L GND #PWR042
+L GND #PWR041
 U 1 1 5492AE1B
 P 1950 1550
-F 0 "#PWR042" H 1950 1550 30  0001 C CNN
+F 0 "#PWR041" H 1950 1550 30  0001 C CNN
 F 1 "GND" H 1950 1480 30  0001 C CNN
 F 2 "" H 1950 1550 60  0000 C CNN
@@
 $EndComp
 $Comp
-L +5V #PWR043
+L +5V #PWR042
 U 1 1 5492AF34
 P 1900 1250
-F 0 "#PWR043" H 1900 1340 20  0001 C CNN
+F 0 "#PWR042" H 1900 1340 20  0001 C CNN
 F 1 "+5V" H 1900 1340 30  0000 C CNN
 F 2 "" H 1900 1250 60  0000 C CNN
@@
 $EndComp
 $Comp
-L +3.3V #PWR044
+L +3.3V #PWR043
 U 1 1 5492AF4D
 P 1900 1350
-F 0 "#PWR044" H 1900 1310 30  0001 C CNN
+F 0 "#PWR043" H 1900 1310 30  0001 C CNN
 F 1 "+3.3V" H 1900 1460 30  0000 C CNN
 F 2 "" H 1900 1350 60  0000 C CNN
@@
 $EndComp
 $Comp
-L +BATT #PWR045
+L +BATT #PWR044
 U 1 1 5492B190
 P 2000 1100
-F 0 "#PWR045" H 2000 1050 20  0001 C CNN
+F 0 "#PWR044" H 2000 1050 20  0001 C CNN
 F 1 "+BATT" H 2000 1200 30  0000 C CNN
 F 2 "" H 2000 1100 60  0000 C CNN
@@
 	3250 4800 3250 5600
 Wire Wire Line
-	3250 5600 2150 5600
-Wire Wire Line
 	3550 4700 3150 4700
 Wire Wire Line
 	3150 4700 3150 5500
-Wire Wire Line
-	3150 5500 2150 5500
 Wire Wire Line
 	2150 5400 3050 5400
@@
 	7200 2300 7200 1050
 Wire Wire Line
-	7200 1050 7950 1050
-Wire Wire Line
 	6650 3300 6750 3300
 Wire Wire Line
@@
 	8050 5350 8050 5300
 Wire Wire Line
-	9300 5300 8050 5300
-Wire Wire Line
-	9300 4700 9300 5300
+	8050 5300 9300 5300
+Wire Wire Line
+	9300 5300 9300 4700
 Wire Wire Line
 	5850 6200 5850 6100
@@
 	7150 5250 7150 6100
 Connection ~ 6550 6100
+$Comp
+L R R11
+U 1 1 54943426
+P 7550 1050
+F 0 "R11" V 7630 1050 40  0000 C CNN
+F 1 "0" V 7557 1051 40  0000 C CNN
+F 2 "~" V 7480 1050 30  0000 C CNN
+F 3 "~" H 7550 1050 30  0000 C CNN
+	1    7550 1050
+	0    -1   -1   0
+$EndComp
+Wire Wire Line
+	7200 1050 7300 1050
+Wire Wire Line
+	7800 1050 7950 1050
+$Comp
+L R R13
+U 1 1 54943703
+P 2600 5500
+F 0 "R13" V 2680 5500 40  0000 C CNN
+F 1 "0" V 2607 5501 40  0000 C CNN
+F 2 "~" V 2530 5500 30  0000 C CNN
+F 3 "~" H 2600 5500 30  0000 C CNN
+	1    2600 5500
+	0    -1   -1   0
+$EndComp
+$Comp
+L R R14
+U 1 1 54943717
+P 2600 5600
+F 0 "R14" V 2680 5600 40  0000 C CNN
+F 1 "0" V 2607 5601 40  0000 C CNN
+F 2 "~" V 2530 5600 30  0000 C CNN
+F 3 "~" H 2600 5600 30  0000 C CNN
+	1    2600 5600
+	0    -1   -1   0
+$EndComp
+Wire Wire Line
+	2150 5500 2350 5500
+Wire Wire Line
+	2150 5600 2350 5600
+Wire Wire Line
+	3150 5500 2850 5500
+Wire Wire Line
+	3250 5600 2850 5600
 $EndSCHEMATC
