File: schematic/rifle-stm32f103ret6-rev1/rifle.kicad_pcb (KiCad board)
At the start: 2 copper layers, 39 parts, among them K1 Magazine, K2 Sound, K3 IR_LASER, P1 Indication, P10 RFID-RC522-MODULE, P11 NRF24L01, P12 CONN_2, P13 IR_LED, P2 MICROSD-SDIO, P3 Reset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

Commit message: About a half of PCB
Parts:
- added P14: Power_in, PIN_ARRAY_2X1, B.Cu at (124.0, 81.8)
- added P15: Power_out, PIN_ARRAY_4x1, B.Cu at (114.0, 95.8)
- K3, P13, P3, P5, P7: moved to B.Cu
- moved C5 103.8 mm to (144.3, 82.0), turned to 270 degrees
- moved U2 100.5 mm to (136.4, 81.8), turned to 270 degrees
- moved U1 95.5 mm to (152.4, 82.0), turned to 270 degrees
- moved C8 92.7 mm to (157.7, 116.1), turned to 180 degrees
- moved C7 85.7 mm to (147.3, 115.3), turned to 180 degrees
- moved C10 85.4 mm to (142.7, 111.3), turned to 180 degrees
- moved P11 80.2 mm to (185.2, 113.0), turned to 90 degrees
- moved P4 72.2 mm to (116.1, 110.2), turned to 90 degrees
- moved C1 71.1 mm to (128.5, 82.0), turned to 270 degrees
- moved P1 70.5 mm to (125.2, 105.2)
- moved P10 69.8 mm to (152.4, 92.2)
- moved P2 66.8 mm to (173.7, 88.4), turned to 90 degrees
- moved P8 64.9 mm to (125.7, 127.0)
- moved P12 64.7 mm to (129.3, 124.7), turned to 270 degrees
- moved Q2 64.5 mm to (147.3, 121.7)
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Connections:
- C5 pad 1: +3.3V -> +5V
- U2 pad 2: +3.3V -> +5V
Routing:
- net GND: track 0.00 -> 152.1 mm, vias 0 -> 2
- net N-0000057: track 0.00 -> 49.9 mm, vias 0 -> 2
- net N-0000048: track 0.00 -> 45.4 mm, vias 0 -> 2
- net +3.3V: track 0.00 -> 42.9 mm
- net N-0000056: track 0.00 -> 39.4 mm, vias 0 -> 2
- net N-0000047: track 0.00 -> 36.4 mm, vias 0 -> 2
- net N-0000046: track 0.00 -> 28.9 mm, vias 0 -> 2
- net N-0000011: track 0.00 -> 26.9 mm
- net N-0000013: track 0.00 -> 26.2 mm
- net N-0000050: track 0.00 -> 25.5 mm
- net N-0000012: track 0.00 -> 24.2 mm
- net N-0000018: track 0.00 -> 23.7 mm
- net N-0000031: track 0.00 -> 23.5 mm
- net N-0000010: track 0.00 -> 23.5 mm
- net N-0000014: track 0.00 -> 22.7 mm
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Other:
- net class Batt+ added: clearance 0.2, trace_width 1, via_dia 0.889, via_drill 0.635
- net class Default: clearance 0.254 -> 0.2; via_dia 0.889 -> 1.5; via_drill 0.635 -> 1
- rule trace_clearance: 0.254 -> 0.2

Commit message: Some more routing
Parts:
- added R10: 0, SM1206, F.Cu at (134.4, 87.2)
- added R12: 0, SM1206, F.Cu at (169.2, 123.3)
- added R5: 0, SM1206, F.Cu at (169.4, 91.2)
- added R6: 0, SM1206, F.Cu at (159.4, 92.2)
- added R7: 0, SM1206, F.Cu at (166.5, 91.2)
- added R8: 0, SM1206, F.Cu at (164.0, 86.7)
- added R9: 0, SM1206, F.Cu at (169.4, 84.5)
- moved P4 70.0 mm to (186.1, 113.3), turned to 270 degrees
- moved C1 20.8 mm to (149.4, 81.3)
- moved Q1 19.9 mm to (138.9, 113.7), turned to 270 degrees
- moved P12 19.7 mm to (111.0, 132.0), turned to 90 degrees
- moved P11 12.8 mm to (184.9, 125.9)
- moved P15 11.9 mm to (124.1, 89.3)
- moved C5 10.1 mm to (134.2, 80.9)
- moved P14 5.66 mm to (129.3, 79.9)
- moved U2 5.14 mm to (141.5, 81.0)
- moved U1 5.14 mm to (157.5, 81.3)
- moved P8 4.77 mm to (129.9, 124.7), turned to 270 degrees
- moved C7 1.91 mm to (147.2, 117.2)
- moved P7 0.81 mm to (158.2, 99.4)
- moved C8 0.76 mm to (157.7, 115.3)
- moved C2 0.40 mm to (150.0, 88.3)
Connections:
- C1 pad 1: +BATT -> N-0000022
- P10 pad 1: N-0000032 (its old number) -> N-000008
- P10 pad 2: N-0000031 -> N-0000044
- P11 pad 1: GND -> N-0000042
- P2 pad 1: N-0000052 (its old number) -> N-0000046
- P2 pad 3: N-0000054 (its old number) -> N-0000048
- P2 pad 4: +3.3V -> N-0000045
- P5 pad 1: GND -> N-0000042
- U1 pad 3: +BATT -> N-0000022
- U2 pad 3: +BATT -> N-0000022
- U3 pad 50: N-0000032 (its old number) -> N-0000041
- U3 pad 51: N-0000052 (its old number) -> N-0000047
- U3 pad 54: N-0000054 (its old number) -> N-0000065
- U3 pad 55: N-0000031 -> N-0000043
Routing:
- net GND: track 152.1 -> 241.3 mm
- net +3.3V: track 42.9 -> 108.1 mm
- net N-0000034: track 0.00 -> 45.5 mm, vias 0 -> 2
- net N-000006: track 0.00 -> 38.4 mm
- net N-0000035: track 0.00 -> 36.8 mm, vias 0 -> 2
- net N-000004: track 0.00 -> 34.8 mm
- net N-0000063: track 0.00 -> 34.4 mm
- net N-000005: track 0.00 -> 32.6 mm
- net N-000001: track 0.00 -> 30.4 mm
- net N-0000033: track 0.00 -> 28.2 mm
- net N-0000047: track 0.00 -> 27.6 mm
- net N-0000064: track 0.00 -> 26.9 mm
- net N-0000031: track 23.5 -> 0.00 mm
- net N-0000042: track 0.00 -> 22.3 mm
- net N-0000022: track 0.00 -> 21.8 mm
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
Commit message: Rwo wires left
Parts:
- added R11: 0, SM1206, F.Cu at (127.5, 122.3)
- added R13: 0, SM1206, F.Cu at (183.3, 110.5)
- added R14: 0, SM1206, F.Cu at (183.3, 107.8)
- moved Q1 20.0 mm to (123.2, 126.0), turned to 90 degrees
- moved P12 17.3 mm to (127.3, 126.0), turned to 0 degrees
- moved P4 5.57 mm to (181.0, 115.6), turned to 0 degrees
- moved P8 1.92 mm to (131.8, 124.5), turned to 90 degrees
- moved P15 0.18 mm to (124.0, 89.2)
- moved C7 0.18 mm to (147.3, 117.1)
- moved P9 0.13 mm to (182.2, 104.6)
Connections:
- P2 pad 7: N-0000067 -> N-0000042
- P2 pad 8: N-0000066 (its old number) -> N-0000043
- Q1 pad G: N-0000038 (its old number) -> N-0000040
- U3 pad 15: N-0000038 (its old number) -> N-0000064
- U3 pad 39: N-0000067 -> N-0000068
- U3 pad 40: N-0000066 (its old number) -> N-0000059
Routing:
- net GND: track 241.3 -> 391.3 mm
- net +3.3V: track 108.1 -> 246.6 mm, vias 0 -> 4
- net N-000006: track 0.00 -> 74.9 mm, vias 0 -> 2
- net +BATT: track 7.52 -> 77.2 mm, vias 0 -> 2
- net N-000005: track 0.00 -> 66.6 mm, vias 0 -> 2
- net N-0000039: track 0.00 -> 56.5 mm, vias 0 -> 2
- net N-0000067: track 36.4 -> 0.00 mm, vias 2 -> 0
- net N-0000042: track 0.00 -> 31.3 mm
- net N-0000043: track 0.00 -> 30.7 mm
- net N-0000066 (its old number): track 28.9 -> 0.00 mm, vias 2 -> 0
- net N-0000064: track 0.00 -> 27.3 mm
- net N-0000028: track 0.00 -> 26.1 mm
- net N-0000068: track 0.00 -> 23.9 mm
- net N-0000059: track 0.00 -> 23.1 mm
- net N-0000029: track 0.00 -> 21.3 mm
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Other:
- net class Batt+: via_dia 0.889 -> 1.5; via_drill 0.635 -> 1

Commit message: PCB seems done
Routing:
- net +5V: track 27.7 -> 121.9 mm, vias 0 -> 2
- net +3.3V: track 246.6 -> 288.3 mm, vias 4 -> 6
- net N-0000063: track 21.0 -> 22.2 mm
Other:
- board outline added: 83.2 x 62.1 mm
- net class Default: trace_width 0.254 -> 1
