File: schematic/simple-ir-remote-control/simple-ir-remote-control-rev1.1/simple-ir-remote-control.sch (KiCad schematic (older format))
At the start: 24 parts, among them K1 CONN_3, P1 CONN_1, P2 CONN_1, P3 CONN_1, P4 CONN_1, P5 CONN_5, P6 CONN_4, P7 CONN_5, P8 CONN_5, P9 CONN_2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

Commit message: Little fix
Parts:
- added P10: CONN_1, ~, symbol CONN_1
Connections:
- net GND: now also P10.1
Changed lines of the file:
@@
 	0    -1   -1   0
 $EndComp
+$Comp
+L CONN_1 P10
+U 1 1 54F1C7CE
+P 9150 4000
+F 0 "P10" H 9230 4000 40  0000 L CNN
+F 1 "CONN_1" H 9150 4055 30  0001 C CNN
+F 2 "~" H 9150 4000 60  0000 C CNN
+F 3 "~" H 9150 4000 60  0000 C CNN
+	1    9150 4000
+	1    0    0    -1
+$EndComp
+$Comp
+L GND #PWR018
+U 1 1 54F1C7DD
+P 8800 4150
+F 0 "#PWR018" H 8800 4150 30  0001 C CNN
+F 1 "GND" H 8800 4080 30  0001 C CNN
+F 2 "" H 8800 4150 60  0000 C CNN
+F 3 "" H 8800 4150 60  0000 C CNN
+	1    8800 4150
+	1    0    0    -1
+$EndComp
+Wire Wire Line
+	8800 4150 8800 4000
+Wire Wire Line
+	8800 4000 9000 4000
 $EndSCHEMATC
