File: schematic/sensor-module/sensor-module.kicad_pcb (KiCad board)
At the start: 2 copper layers, 27.3 x 24.3 mm, 14 parts, among them K1 SENSORS, K2 LEDs, K3 SENSORS, K4 LEDs, P1 Vibro, P2 VibroEngine, P3 Vibro, U1 RGB-LED

Commit message: sensor module pcb fixed for vibroengine
Parts:
- moved R7 2.19 mm to (40.4, 42.9), turned to 270 degrees
Connections:
- P1 pad 1: N-0000015 (its old number) -> N-0000013
- P2 pad 1: GND -> N-0000013
- P3 pad 1: N-0000015 (its old number) -> N-0000013
- R7 pad 2: N-0000015 (its old number) -> +BATT
Routing:
- net N-0000015 (its old number): track 24.9 -> 0.00 mm
- net N-0000013: track 0.00 -> 24.2 mm
- net GND: track 58.0 -> 55.9 mm
- net +BATT: track 29.0 -> 30.5 mm
