File: schematic/rifle/rifle-shield-v1-rev1/rifle-shield-v1.sch (KiCad schematic (older format))
At the start: 9 parts

Commit message: rifle shield done without indication
Parts:
- added C?: 0.1uF, ~, symbol C
- added C?: 470uF, ~, symbol CP1
- added C? (x3): 1uF, ~, symbol C
- added C? (x2): 0.47uF, ~, symbol C
- added C?: C, ~, symbol C
- added K?: LASER, ~, symbol CONN_3
- added P?: Speaker1, ~, symbol CONN_2
- added P?: Speaker2, ~, symbol CONN_2
- added P?: Mag&fireMode, ~, symbol CONN_4
- added P?: Fire&Reload, ~, symbol CONN_2
- added P?: IR_LED, ~, symbol CONN_2
- added P?: USART1, ~, symbol CONN_4
- added P?: CONN_2, ~, symbol CONN_2
- added P?: Vibro&flash, ~, symbol CONN_2
- added Q? (x6): MOS_N, ~, symbol MOS_N
- added Q?: MOSFET_P, ~, symbol MOSFET_P
- added R? (x9): R, ~, symbol R
- added U?: PAM8403, ~, symbol PAM8403
Connections:
- net GND: now also C?.1, C?.2, C?.2, C?.2, C?.2, C?.2, K?.2 (PM), P?.1 (P1), P?.1 (P1), P?.1 (P1), Q?.G, Q?.S, Q?.S, Q?.S, Q?.S, Q?.S, Q?.S, R?.2, U?.11 (GND), U?.15 (PGND), U?.2 (PGND), U?.9 (NC)
- net VCC: now also K?.1 (P1), Q?.S, R?.1
- net at P?.10 (P10): now also Q?.G
- net at P?.11 (P11): now also Q?.G
- net at P?.12 (P12): now also R?.2
- net at P?.14 (P14): now also Q?.G
- net at P?.15 (P15): now also K?.3 (P3), Q?.G
- net at P?.16 (P16): now also R?.1, R?.2
- net at P?.18 (P18): now also Q?.G
- net at P?.19 (P19): now also Q?.G
- net at P?.4 (P4): now also P?.1 (P1)
- net at P?.5 (P5): now also P?.2 (P2)
- net at P?.6 (P6): now also P?.3 (P3)
- net at P?.7 (P7): now also P?.4 (P4)
- net at P?.8 (P8): now also P?.1 (P1)
- net at P?.9 (P9): now also P?.2 (PM)
- net at P?.10 (P10): now also P?.4 (P4)
- net at P?.9 (P9): now also P?.3 (P3)
- new net: P?.2 (PM), U?.1 (+OutLeft)
- new net: R?.2, U?.10 (InRight)
- new net: C?.1, C?.1, C?.1, C?.1, U?.12 (~Shutdown), U?.13 (PVDD), U?.4 (PVDD), U?.5 (~Mute), U?.6 (VDD)
- new net: P?.1 (P1), U?.14 (-OutRight)
- new net: P?.2 (PM), U?.16 (+OutRight)
- new net: P?.1 (P1), U?.3 (-OutLeft)
- new net: R?.2, U?.7 (InLeft)
- new net: C?.2, U?.8 (Vref)
- new net: C?.2, R?.1 (x2)
- new net: C?.1, C?.1, C?.1, R?.1
- new net: Q?.D, R?.1 (x4)
- new net: P?.2 (PM), R?.2, R?.2, R?.2, R?.2
- new net: P?.2 (PM), Q?.D (x2)
- new net: P?.1 (P1), Q?.D
Other:
- moved on the sheet: BT?, C?, U?

Commit message: rifle shield PCB beginned :/
Parts:
- removed BT?: BATTERY, ~, symbol BATTERY
- added K1: Display2, ~, symbol CONN_3
- added K3: VCC, ~, symbol CONN_3
- added P8: GND, ~, symbol CONN_5
- added P9: Display1, ~, symbol CONN_7
- P1: renamed from P?; value CONN_2 -> Power
- gave numbers to parts that had none: 41
Connections:
- net GND: now also P8.1, P8.2, P8.3, P8.4, P8.5; no longer P13.1 (P1)
- net VCC: now also C11.1, C6.1, C8.1, C9.1, P13.2 (PM), U1.12 (~Shutdown), U1.13 (PVDD), U1.4 (PVDD), U1.5 (~Mute), U1.6 (VDD), K3.1 (P1), K3.2 (PM), K3.3 (P3)
- net at P2.13 (P13): now also K1.1 (P1)
- net at P2.17 (P17): now also K1.2 (PM)
- net at P2.20 (P20): now also K1.3 (P3)
- net at P10.1 (P1): now also P9.1 (P1)
- net at P10.11 (P11): now also P9.5 (P5)
- net at P10.12 (P12): now also P9.6 (P6)
- net at P10.2 (P2): now also P9.2 (P2)
- net at P10.20 (P20): now also P9.7 (P7)
- net at P10.7 (P7): now also P9.3 (P3)
- net at P10.8 (P8): now also P9.4 (P4)
- net at R6.2, R7.2, R8.2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: now also P13.1 (P1); no longer P13.2 (PM)
Other:
- moved on the sheet: P13, P6
