File: schematic/head-sensor/head-sensor-shield-v1-rev1/head-sensor-shield-v1-rev1.sch (KiCad schematic (older format))
At the start: 24 parts

Commit message: Head sensor shield done
Parts:
- added K5: 3.3 V, ~, symbol CONN_3
- C1: renamed from C?; value C -> 1uF
- C2, C3: renamed from C?; value CP1 -> 100uF
- gave numbers to parts that had none: 21
Connections:
- net +3.3V: now also K5.1 (P1), K5.2 (PM), K5.3 (P3)
- net at P3.14 (P14): now also Q2.G
- net at P3.15 (P15): now also Q3.G
- net at P3.18 (P18): now also Q4.G; no longer Q2.G
- net at P3.19 (P19): no longer Q3.G
- net at P3.20 (P20): no longer Q4.G
