File: schematic/head-sensor/head-sensor-shield-v1-rev1/head-sensor-shield-v1-rev1.kicad_pcb (KiCad board)
At the start: 2 copper layers, 50 x 25.9 mm, 26 parts, among them K1 GND, K2 Sensors_in, K3 RGB_leds, K4 Vibro, K5 3.3 V, P1 Power_in, P2 VCC, P3 MCU1, P4 USART1, P6 MCU2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

Commit message: PCB: MCU2 connector orientation fixed; SOFT: Worker object added to os-wrappers, WavPlayer and IOPinsPool use it now
Parts:
- moved P8 20.5 mm to (96.8, 69.3)
- moved P7 20.3 mm to (96.7, 49.0)
- turned P4 to 270 degrees
- turned P6 to 90 degrees
Routing:
- net GND: track 37.6 -> 53.4 mm, vias 12 -> 14
- net N-0000025: track 6.21 -> 16.0 mm
- net N-0000043: track 6.41 -> 16.2 mm
- net N-0000037: track 33.9 -> 25.1 mm, vias 1 -> 0
- net N-0000027: track 16.2 -> 8.82 mm
- net N-0000026: track 8.23 -> 15.1 mm
- net N-0000045: track 6.61 -> 12.5 mm
- net N-0000048: track 8.62 -> 3.00 mm
- net N-0000044: track 8.60 -> 3.92 mm
- net N-0000024: track 11.1 -> 6.95 mm
- net N-0000047: track 4.02 -> 6.60 mm
- net N-0000046: track 11.5 -> 9.03 mm
- net +3.3V: track 75.3 -> 77.1 mm
- net VCC: track 50.3 -> 51.1 mm, vias 4 -> 2
- net N-0000038: track 25.3 -> 24.6 mm
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Other:
- board text added: "Caustic LT system head sensor shield v1 3c rev.2"
