File: schematic/head-sensor/head-sensor-shield-v2-rev1/head-sensor-shield-v2-rev1.kicad_pcb (KiCad board)
At the start: 2 copper layers, 50 x 26.2 mm, 23 parts, among them P1 Power_in, P2 Zone2, P3 MCU1, P4 USART1, P6 MCU2, P7 RFID, P8 NRF24L01, P9 Zone1, Q1 IRLML6402, Q5 IRLML2502 x 5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

Commit message: MCU module rev2 done
Parts:
- added P5: UART3, PIN_ARRAY_4x1, B.Cu at (110.9, 65.5)
- +: renamed from + BT1
- P4: value USART1 -> UART1
- Q1: value IRLML6402 -> (none)
- Q5: value IRLML2502 x 5 -> IRLML2502
- U1: footprint sot323-5 -> sot323-5-fx
- moved P4 3.90 mm to (110.9, 52.7)
- moved U1 0.10 mm to (98.2, 54.1)
Routing:
- net GND: track 30.3 -> 75.3 mm, vias 9 -> 16
- net +3.3V: track 104.5 -> 124.6 mm, vias 4 -> 5
- net N-0000015: track 0.00 -> 7.59 mm
- net N-000004: track 0.00 -> 4.00 mm
- net N-0000024: track 7.17 -> 10.1 mm
- net N-0000023: track 3.61 -> 6.08 mm
- net (no net): track 0.30 -> 0.00 mm, vias 12 -> 0
