File: schematic/sensor-module/sensor-module-idc/sensor-module.kicad_pcb (KiCad board)
At the start: 2 copper layers, 46.2 x 43.5 mm, 40 parts, among them P1 SENSOR_CONNECTOR, P2 VibroEngine, U2 RGB-LED, U3 TSOP4856

Commit message: Head and rifle boards done
Parts:
- removed the ? at (93.4, 61.9)
- removed the ? at (93.4, 76.6)
- removed the ? at (93.4, 53.6)
- removed the ? at (93.4, 38.9)
- removed the ? at (85.5, 76.5)
- removed the ? at (85.5, 61.8)
- removed P1 (x4): SENSOR_CONNECTOR, Sensors-connector-10x
- removed the P2 at (107.8, 77.4)
- removed the P2 at (107.8, 54.4)
- removed the P2 at (71.1, 61.0)
- removed the R4 at (99.9, 70.9)
- removed the R4 at (99.9, 47.9)
- removed the R4 at (79.0, 67.5)
- removed the R5 at (99.9, 73.3)
- removed the R5 at (99.9, 50.3)
- removed the R5 at (79.0, 65.1)
- removed the R6 at (99.9, 75.9)
- removed the R6 at (99.9, 52.9)
- removed the R6 at (79.0, 62.5)
- removed the R7 at (101.7, 77.5)
- removed the R7 at (101.7, 54.5)
- removed the R7 at (77.2, 60.9)
- removed the U2 at (101.7, 73.5)
- removed the U2 at (101.7, 50.5)
- removed the U2 at (77.2, 64.9)
- removed the U3 at (105.7, 65.0)
- removed the U3 at (105.7, 42.0)
- removed the U3 at (73.2, 73.4)
Routing:
- net +BATT: track 117.5 -> 29.4 mm, vias 4 -> 1
- net N-0000013: track 38.6 -> 9.65 mm, vias 4 -> 1
- net N-0000014: track 36.6 -> 9.16 mm
- net N-000007: track 34.9 -> 8.72 mm
- net N-0000012: track 32.3 -> 8.09 mm
- net N-000003: track 31.4 -> 7.86 mm
- net +3.3V: track 20.4 -> 5.09 mm
- net GND: track 20.4 -> 5.09 mm
- net N-000006: track 19.6 -> 4.90 mm, vias 4 -> 1
- net N-000004: track 19.3 -> 4.82 mm, vias 4 -> 1
- net N-000005: track 18.1 -> 4.53 mm, vias 4 -> 1
- net N-000008: track 12.9 -> 3.22 mm
Other:
- board outline removed

Commit message: Group made
Parts:
- added P1: SENSOR_CONNECTOR, Sensors-connector-10x, F.Cu at (68.5, 46.5)
Changed lines of the file:
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@@
 (kicad_pcb (version 3) (host pcbnew "(2013-may-18)-stable")
   (general
-    (links 15)
-    (no_connects 0)
-    (area 57.020999 34.813 121.854001 80.562)
+    (links 18)
+    (no_connects 3)
+    (area 0 0 0 0)
     (thickness 1.6)
     (drawings 1)
     (tracks 60)
     (zones 0)
-    (modules 9)
-    (nets 13)
+    (modules 10)
+    (nets 16)
   )
   (page A3)
@@
   (net 5 N-0000013)
   (net 6 N-0000014)
-  (net 7 N-000003)
-  (net 8 N-000004)
-  (net 9 N-000005)
-  (net 10 N-000006)
-  (net 11 N-000007)
-  (net 12 N-000008)
+  (net 7 N-0000015)
+  (net 8 N-0000016)
+  (net 9 N-0000017)
+  (net 10 N-000003)
+  (net 11 N-000004)
+  (net 12 N-000005)
+  (net 13 N-000006)
+  (net 14 N-000007)
+  (net 15 N-000008)
   (net_class Default "This is the default net class."
     (clearance 0.254)
@@
     (add_net N-0000013)
     (add_net N-0000014)
+    (add_net N-0000015)
+    (add_net N-0000016)
+    (add_net N-0000017)
     (add_net N-000003)
     (add_net N-000004)
@@
     (pad 2 smd rect (at 1.651 0) (size 1.524 2.032)
       (layers B.Cu B.Paste B.Mask)
-      (net 10 N-000006)
+      (net 13 N-000006)
     )
     (model smd/chip_cms.wrl
@@
     (pad 2 smd rect (at 1.651 0) (size 1.524 2.032)
       (layers B.Cu B.Paste B.Mask)
-      (net 9 N-000005)
+      (net 12 N-000005)
     )
     (model smd/chip_cms.wrl
@@
     (pad 2 smd rect (at 1.651 0) (size 1.524 2.032)
       (layers B.Cu B.Paste B.Mask)
-      (net 8 N-000004)
+      (net 11 N-000004)
     )
     (model smd/chip_cms.wrl
@@
     (pad 1 smd rect (at -1.651 0) (size 1.524 2.032)
       (layers F.Cu F.Paste F.Mask)
-      (net 12 N-000008)
+      (net 15 N-000008)
     )
     (pad 2 smd rect (at 1.651 0) (size 1.524 2.032)
@@
     (pad 4 smd rect (at -2.5 -1.5 180) (size 2 1)
       (layers F.Cu F.Paste F.Mask)
-      (net 10 N-000006)
+      (net 13 N-000006)
     )
     (pad 5 smd rect (at -2.5 0 180) (size 2 1)
       (layers F.Cu F.Paste F.Mask)
-      (net 9 N-000005)
+      (net 12 N-000005)
     )
     (pad 6 smd rect (at -2.5 1.5 180) (size 2 1)
       (layers F.Cu F.Paste F.Mask)
-      (net 8 N-000004)
+      (net 11 N-000004)
     )
   )
@@
     (pad 1 thru_hole rect (at -2.54 0 90) (size 2 2.5) (drill 1)
       (layers *.Cu *.Mask F.SilkS)
-      (net 7 N-000003)
+      (net 10 N-000003)
     )
     (pad 2 thru_hole oval (at 0 0 90) (size 2 2.5) (drill 1)
@@
     (pad 1 thru_hole rect (at -1.27 0 180) (size 2 2.5) (drill 1)
       (layers *.Cu *.Mask F.SilkS)
-      (net 12 N-000008)
+      (net 15 N-000008)
     )
     (pad 2 thru_hole oval (at 1.27 0 180) (size 2 2.5) (drill 1)
       (layers *.Cu *.Mask F.SilkS)
-      (net 11 N-000007)
+      (net 14 N-000007)
     )
   )
@@
     (pad 1 thru_hole circle (at 0 0) (size 4.064 4.064) (drill 3)
       (layers *.Cu *.Mask F.SilkS)
+    )
+  )
+  (module Sensors-connector-10x (layer F.Cu)
+    (at 68.4784 46.482)
+    (fp_text reference P1 (at -3.5 0 90) (layer F.SilkS)
+      (effects (font (size 1 1) (thickness 0.15)))
+    )
+    (fp_text value SENSOR_CONNECTOR (at -5.75 0 90) (layer F.SilkS)
+      (effects (font (size 1 1) (thickness 0.15)))
+    )
+    (fp_line (start -11.25 -2.5) (end -4.5 -2.5) (layer F.SilkS) (width 0.15))
+    (fp_line (start -4.5 -2.5) (end -4.5 2.5) (layer F.SilkS) (width 0.15))
+    (fp_line (start -4.5 2.5) (end -11.25 2.5) (layer F.SilkS) (width 0.15))
+    (fp_line (start -2.5 -10) (end -2.5 10) (layer F.SilkS) (width 0.15))
+    (fp_line (start -2.5 10) (end -11.25 10) (layer F.SilkS) (width 0.15))
+    (fp_line (start -11.25 10) (end -11.25 -10) (layer F.SilkS) (width 0.15))
+    (fp_line (start -11.25 -10) (end -2.5 -10) (layer F.SilkS) (width 0.15))
+    (pad 5 smd rect (at 0 0) (size 3.5 2)
+      (layers *.Mask F.Cu F.Paste)
+      (net 4 N-0000012)
+    )
+    (pad 7 smd rect (at 0 -2.54) (size 3.5 2)
+      (layers *.Mask F.Cu F.Paste)
+      (net 6 N-0000014)
+    )
+    (pad 9 smd rect (at 0 -5.08) (size 3.5 2)
+      (layers *.Mask F.Cu F.Paste)
+    )
+    (pad 3 smd rect (at 0 2.54) (size 3.5 2)
+      (layers *.Mask F.Cu F.Paste)
+      (net 1 +3.3V)
+    )
+    (pad 1 smd rect (at 0 5.08) (size 3.5 2)
+      (layers *.Mask F.Cu F.Paste)
+      (net 3 GND)
+    )
+    (pad 2 smd rect (at 0 5.08) (size 3.5 2)
+      (layers *.Mask B.Cu F.Paste)
+      (net 2 +BATT)
+    )
+    (pad 4 smd rect (at 0 2.54) (size 3.5 2)
+      (layers *.Mask B.Cu F.Paste)
+      (net 10 N-000003)
+    )
+    (pad 6 smd rect (at 0 0) (size 3.5 2)
+      (layers *.Mask B.Cu F.Paste)
+      (net 5 N-0000013)
+    )
+    (pad 8 smd rect (at 0 -2.54) (size 3.5 2)
+      (layers *.Mask B.Cu F.Paste)
+      (net 14 N-000007)
+    )
+    (pad 10 smd rect (at 0 -5.08) (size 3.5 2)
+      (layers *.Mask B.Cu F.Paste)
     )
   )
@@
   (segment (start 71.1 43.5) (end 71.1 40.8) (width 0.6) (layer F.Cu) (net 6))
   (segment (start 70.64 43.96) (end 71.1 43.5) (width 0.6) (layer F.Cu) (net 6))
-  (segment (start 68.6 49.04) (end 70.44 49.04) (width 0.6) (layer B.Cu) (net 7))
-  (segment (start 70.44 49.04) (end 71.1 49.7) (width 0.6) (layer B.Cu) (net 7))
-  (segment (start 71.1 49.7) (end 71.1 52.5) (width 0.6) (layer B.Cu) (net 7))
-  (segment (start 71.1 52.5) (end 71.54 52.94) (width 0.6) (layer B.Cu) (net 7))
-  (segment (start 71.54 52.94) (end 73.2 52.94) (width 0.6) (layer B.Cu) (net 7))
-  (segment (start 80.651 39.5) (end 82.4 39.5) (width 0.6) (layer B.Cu) (net 8))
-  (segment (start 81.5 40.4) (end 79.7 40.4) (width 0.6) (layer F.Cu) (net 8))
-  (segment (start 82.4 39.5) (end 81.5 40.4) (width 0.6) (layer F.Cu) (net 8))
-  (via (at 82.4 39.5) (size 0.7) (layers F.Cu B.Cu) (net 8))
-  (segment (start 79.7 41.9) (end 82.4 41.9) (width 0.6) (layer F.Cu) (net 9))
-  (segment (start 82.2 42.1) (end 80.651 42.1) (width 0.6) (layer B.Cu) (net 9))
-  (segment (start 82.4 41.9) (end 82.2 42.1) (width 0.6) (layer B.Cu) (net 9))
-  (via (at 82.4 41.9) (size 0.7) (layers F.Cu B.Cu) (net 9))
-  (segment (start 80.651 44.5) (end 82.3 44.5) (width 0.6) (layer B.Cu) (net 10))
-  (segment (start 81.4 43.4) (end 79.7 43.4) (width 0.6) (layer F.Cu) (net 10))
-  (segment (start 82.4 44.4) (end 81.4 43.4) (width 0.6) (layer F.Cu) (net 10))
-  (via (at 82.4 44.4) (size 0.7) (layers F.Cu B.Cu) (net 10))
-  (segment (start 82.3 44.5) (end 82.4 44.4) (width 0.6) (layer B.Cu) (net 10))
-  (segment (start 68.6 43.96) (end 70.64 43.96) (width 0.6) (layer B.Cu) (net 11))
-  (segment (start 69.83 39.03) (end 69.83 38) (width 0.6) (layer B.Cu) (net 11))
-  (segment (start 71.1 40.3) (end 69.83 39.03) (width 0.6) (layer B.Cu) (net 11))
-  (segment (start 71.1 43.5) (end 71.1 40.3) (width 0.6) (layer B.Cu) (net 11))
-  (segment (start 70.64 43.96) (end 71.1 43.5) (width 0.6) (layer B.Cu) (net 11))
-  (segment (start 72.37 38) (end 75.449 38) (width 0.6) (layer F.Cu) (net 12))
-  (segment (start 75.449 38) (end 75.549 37.9) (width 0.6) (layer F.Cu) (net 12))
+  (segment (start 68.6 49.04) (end 70.44 49.04) (width 0.6) (layer B.Cu) (net 10))
+  (segment (start 70.44 49.04) (end 71.1 49.7) (width 0.6) (layer B.Cu) (net 10))
+  (segment (start 71.1 49.7) (end 71.1 52.5) (width 0.6) (layer B.Cu) (net 10))
+  (segment (start 71.1 52.5) (end 71.54 52.94) (width 0.6) (layer B.Cu) (net 10))
+  (segment (start 71.54 52.94) (end 73.2 52.94) (width 0.6) (layer B.Cu) (net 10))
+  (segment (start 80.651 39.5) (end 82.4 39.5) (width 0.6) (layer B.Cu) (net 11))
+  (segment (start 81.5 40.4) (end 79.7 40.4) (width 0.6) (layer F.Cu) (net 11))
+  (segment (start 82.4 39.5) (end 81.5 40.4) (width 0.6) (layer F.Cu) (net 11))
+  (via (at 82.4 39.5) (size 0.7) (layers F.Cu B.Cu) (net 11))
+  (segment (start 79.7 41.9) (end 82.4 41.9) (width 0.6) (layer F.Cu) (net 12))
+  (segment (start 82.2 42.1) (end 80.651 42.1) (width 0.6) (layer B.Cu) (net 12))
+  (segment (start 82.4 41.9) (end 82.2 42.1) (width 0.6) (layer B.Cu) (net 12))
+  (via (at 82.4 41.9) (size 0.7) (layers F.Cu B.Cu) (net 12))
+  (segment (start 80.651 44.5) (end 82.3 44.5) (width 0.6) (layer B.Cu) (net 13))
+  (segment (start 81.4 43.4) (end 79.7 43.4) (width 0.6) (layer F.Cu) (net 13))
+  (segment (start 82.4 44.4) (end 81.4 43.4) (width 0.6) (layer F.Cu) (net 13))
+  (via (at 82.4 44.4) (size 0.7) (layers F.Cu B.Cu) (net 13))
+  (segment (start 82.3 44.5) (end 82.4 44.4) (width 0.6) (layer B.Cu) (net 13))
+  (segment (start 68.6 43.96) (end 70.64 43.96) (width 0.6) (layer B.Cu) (net 14))
+  (segment (start 69.83 39.03) (end 69.83 38) (width 0.6) (layer B.Cu) (net 14))
+  (segment (start 71.1 40.3) (end 69.83 39.03) (width 0.6) (layer B.Cu) (net 14))
+  (segment (start 71.1 43.5) (end 71.1 40.3) (width 0.6) (layer B.Cu) (net 14))
+  (segment (start 70.64 43.96) (end 71.1 43.5) (width 0.6) (layer B.Cu) (net 14))
+  (segment (start 72.37 38) (end 75.449 38) (width 0.6) (layer F.Cu) (net 15))
+  (segment (start 75.449 38) (end 75.549 37.9) (width 0.6) (layer F.Cu) (net 15))
 )
