File: schematic/head-sensor/head-sensor-shield-v3-rev1/head-sensor-shield.sch (KiCad schematic (older format))
At the start: 35 parts, among them K1 Power, P1 USB, P2 Zone2, P3 MCU1, P4 USART1, P5 EXTENSION-CONNECTOR, P6 MCU2, P8 NRF24L01, P9 Zone1, Q1 MOSFET_P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

Commit message: Some job for registering unknown commads
Connections:
- wire segments 195 -> 196
Changed lines of the file:
@@
 Sheet 1 1
 Title "Head sensor shield"
-Date "21 jan 2016"
+Date "14 feb 2016"
 Rev "3.1"
 Comp ""
@@
 	6600 2550 5700 2550
 Connection ~ 5700 2550
+$Comp
+L GND #PWR?
+U 1 1 56C0AB66
+P 1650 10600
+F 0 "#PWR?" H 1650 10600 30  0001 C CNN
+F 1 "GND" H 1650 10530 30  0001 C CNN
+F 2 "" H 1650 10600 60  0000 C CNN
+F 3 "" H 1650 10600 60  0000 C CNN
+	1    1650 10600
+	1    0    0    -1
+$EndComp
+Wire Wire Line
+	1650 10500 1650 10600
 $EndSCHEMATC
