File: schematic/ir-led-module/ir-led-round-lw-compatible/ir-led-lw-compatible.kicad_pcb (KiCad board)
At the start: 2 copper layers, 41.9 x 42.1 mm, 45 parts, among them P1 IR, P2 LIGHT, P3 VCC

Commit message: [PCB] Fix for prev commit
Parts:
- moved D1 72.7 mm to (64.1, 38.2)
- moved D1 72.7 mm to (40.8, 37.0)
- moved D1 72.7 mm to (62.7, 61.4)
- moved D1 72.7 mm to (39.4, 60.3)
- moved D2 72.7 mm to (67.0, 34.0)
- moved D2 72.7 mm to (36.6, 34.1)
- moved D2 72.7 mm to (66.9, 64.3)
- moved D2 72.7 mm to (36.5, 64.5)
- moved D3 72.7 mm to (67.0, 42.4)
- moved D3 72.7 mm to (45.0, 34.1)
- moved D3 72.7 mm to (58.5, 64.3)
- moved D3 72.7 mm to (36.5, 56.1)
- moved D4 72.7 mm to (58.6, 42.4)
- moved D4 72.7 mm to (45.0, 42.5)
- moved D4 72.7 mm to (58.5, 55.9)
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