File: schematic/sensor-module/sensor-tube/sensor-tube.sch (KiCad schematic (older format))
At the start: 7 parts, among them P1 SENSOR_CONNECTOR, U1 RGB-LED, U2 TSOP4856

Commit message: [PCB] Fix for tube sensor
Parts:
- P1: footprint (none) -> components:caustic-sensors-tube-connector
- P2: renamed from P?; footprint (none) -> components:caustic-sensors-tube-connector
- R1, R2, R3: footprint (none) -> Resistors_SMD:R_0805
- U1: footprint (none) -> LEDs:LED_WS2812-PLCC6
- U2: footprint (none) -> Pin_Headers:Pin_Header_Straight_1x03
Changed lines of the file:
@@
 F 0 "U1" H 6000 1750 60  0000 C CNN
 F 1 "RGB-LED" H 6000 2550 60  0000 C CNN
-F 2 "" H 6000 2100 60  0000 C CNN
+F 2 "LEDs:LED_WS2812-PLCC6" H 6000 2100 60  0001 C CNN
 F 3 "" H 6000 2100 60  0000 C CNN
 	1    6000 2150
@@
 F 0 "P1" H 4250 1950 60  0000 C CNN
 F 1 "SENSOR_CONNECTOR" H 4250 2750 60  0000 C CNN
-F 2 "" H 4250 2450 60  0000 C CNN
+F 2 "components:caustic-sensors-tube-connector" H 4250 2450 60  0001 C CNN
 F 3 "" H 4250 2450 60  0000 C CNN
 	1    4150 2200
@@
 F 0 "R1" V 7030 1950 50  0000 C CNN
 F 1 "200" V 6950 1950 50  0000 C CNN
-F 2 "" V 6880 1950 50  0000 C CNN
+F 2 "Resistors_SMD:R_0805" V 6880 1950 50  0001 C CNN
 F 3 "" H 6950 1950 50  0000 C CNN
 	1    6950 1950
@@
 F 0 "R2" V 7030 2150 50  0000 C CNN
 F 1 "150" V 6950 2150 50  0000 C CNN
-F 2 "" V 6880 2150 50  0000 C CNN
+F 2 "Resistors_SMD:R_0805" V 6880 2150 50  0001 C CNN
 F 3 "" H 6950 2150 50  0000 C CNN
 	1    6950 2150
@@
 F 0 "R3" V 7030 2350 50  0000 C CNN
 F 1 "150" V 6950 2350 50  0000 C CNN
-F 2 "" V 6880 2350 50  0000 C CNN
+F 2 "Resistors_SMD:R_0805" V 6880 2350 50  0001 C CNN
 F 3 "" H 6950 2350 50  0000 C CNN
 	1    6950 2350
@@
 F 0 "U2" H 7950 2600 60  0000 C CNN
 F 1 "TSOP4856" H 8000 1850 60  0000 C CNN
-F 2 "" H 8000 2250 60  0000 C CNN
+F 2 "Pin_Headers:Pin_Header_Straight_1x03" H 8000 2250 60  0001 C CNN
 F 3 "" H 8000 2250 60  0000 C CNN
 	1    8000 2250
@@
 	7800 2650 7800 2550
 $Comp
-L SENSOR_CONNECTOR P?
+L SENSOR_CONNECTOR P2
 U 1 1 583C8034
 P 4150 4300
-F 0 "P?" H 4250 4050 60  0000 C CNN
+F 0 "P2" H 4250 4050 60  0000 C CNN
 F 1 "SENSOR_CONNECTOR" H 4250 4850 60  0000 C CNN
-F 2 "" H 4250 4550 60  0000 C CNN
+F 2 "components:caustic-sensors-tube-connector" H 4250 4550 60  0001 C CNN
 F 3 "" H 4250 4550 60  0000 C CNN
 	1    4150 4300
@@
 	5100 3100 4850 3100
 $Comp
-L GND #PWR?
+L GND #PWR03
 U 1 1 583C855B
 P 5100 5050
-F 0 "#PWR?" H 5100 4800 50  0001 C CNN
+F 0 "#PWR03" H 5100 4800 50  0001 C CNN
 F 1 "GND" H 5100 4900 50  0000 C CNN
 F 2 "" H 5100 5050 50  0000 C CNN
