File: schematic/grouped-boards/rifle-sensors/rifle-and-sensors.kicad_pcb (KiCad board)
At the start: 2 copper layers, 93.9 x 97.8 mm, 268 parts, among them P1 BUS, P1 MICROSD-SDIO-CD, P10 RC522, P11 Speaker1, P12 Speaker2, P13 I2C display, P14 I2C display, P15 FLASH, P16 VIBRO, P17 IR_LED, P18 USB_OTG, P19 GND, P2 BUS, P2 SWD, P20 TTL, P3 G B Vcc, P3 SWD, P4 NRF24L01, P4 PA0, P5 PA1, P5 USB_A, P6 PA3, P6 S_A_M1_M2, P7 DEBUG_TX, P7 PA10, P8 Fire, P8 V+, P9 Reload, P9 V-, Q1 IRLML6402, Q1 Q_NMOS_GSD, Q2 IRLML2502, Q2 Q_NMOS_GSD, Q3 IRLML2502, Q3 Q_NMOS_GSD, Q4 IRLML2502, Q5 IRLML2502, Q6 IRLML2502, Q7 IRLML2502, T1 TSOP4856, U1 NCP551, U1 STM32F103RE, U2 STM32F030F4Px, U2 USBLC6-4, U3 MCP73831, U3 RGB, U3 RGB-LED, U4 NCP551, U5 PAM8403, Y1 8MHz

Commit message: Grouped board with rifle and smart sensors fixed
Parts:
- removed the P7 at (85.6, 103.7)
- removed the P7 at (50.3, 103.7)
- removed the R1 at (66.9, 107.1)
- removed the R1 at (31.5, 107.1)
- removed the R5 at (82.0, 99.1)
- removed the R5 at (46.7, 99.1)
- removed the R8 at (82.5, 100.1)
- removed the R8 at (47.2, 100.1)
- removed the REF** at (28.1, 103.8)
- removed the REF** at (46.1, 103.8)
- added P7: PA10, Pin_Headers:Pin_Header_Straight_1x01_Pitch2.54mm, F.Cu at (82.3, 99.5)
- added P7: PA10, Pin_Headers:Pin_Header_Straight_1x01_Pitch2.54mm, F.Cu at (47.1, 99.5)
- added R1: 150, Resistors_SMD:R_0805, F.Cu at (66.3, 108.0)
- added R1: 150, Resistors_SMD:R_0805, F.Cu at (31.1, 108.0)
- added R5: 10k, Resistors_SMD:R_0805, F.Cu at (82.2, 96.1)
- added R5: 10k, Resistors_SMD:R_0805, F.Cu at (47.0, 96.1)
- added R8: R_load, Resistors_SMD:R_0805, B.Cu at (82.3, 96.0)
- added R8: R_load, Resistors_SMD:R_0805, B.Cu at (47.1, 96.0)
- added REF**: 1pin, Connect:1pin, F.Cu at (46.2, 103.8)
- added REF**: 1pin, Connect:1pin, F.Cu at (28.2, 103.8)
- moved C3 0.13 mm to (31.7, 96.4)
- moved C4 0.13 mm to (43.2, 109.4)
- moved D1 0.13 mm to (38.5, 96.5)
- moved P1 0.13 mm to (34.7, 91.8)
- moved P2 0.13 mm to (34.7, 115.8)
- moved P6 0.13 mm to (47.1, 107.6)
- moved P8 0.13 mm to (47.2, 110.8)
- moved P9 0.13 mm to (44.5, 113.6)
- moved Q2 0.13 mm to (43.7, 97.0)
- moved Q3 0.13 mm to (43.5, 97.1)
- moved R6 0.13 mm to (43.5, 93.8)
- moved R7 0.13 mm to (42.9, 93.9)
- moved T1 0.13 mm to (42.0, 106.3)
- moved U1 0.13 mm to (32.1, 97.3)
- moved U2 0.13 mm to (36.3, 103.7)
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Routing:
- net PA10: track 35.6 -> 43.9 mm
- net Net-(P7-Pad1): track 10.4 -> 5.04 mm
- net red: track 36.9 -> 41.6 mm
- net Net-(Q3-Pad3): track 15.1 -> 10.8 mm
- net GND: track 336.7 -> 340.1 mm
- net Net-(R1-Pad1): track 18.2 -> 17.5 mm
